File: PCB/StrainGauge/StrainGauge.kicad_sch (KiCad schematic)
At the start: 0 parts

Commit message: Added first symbol to LIB
Parts:
- added IC1: STM32H523CEU6, QFN50P700X700X60-49N-D, symbol StrainGaugeSYM:STM32H523CEU6
Changed lines of the file:
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@@
     (comment 1 "Author: Mieszko Celiński")
+  )
+  (symbol (lib_id "StrainGaugeSYM:STM32H523CEU6") (at 107.95 49.53 0) (unit 1)
+    (in_bom yes) (on_board yes) (dnp no)
+    (property "Reference" "IC1" (at 104.14 41.91 0)
+      (effects (font (size 1.27 1.27)))
+    )
+    (property "Value" "STM32H523CEU6" (at 104.14 44.45 0)
+      (effects (font (size 1.27 1.27)))
+    )
+    (property "Footprint" "QFN50P700X700X60-49N-D" (at 149.86 134.29 0)
+      (effects (font (size 1.27 1.27)) (justify left top) hide)
+    )
+    (property "Datasheet" "https://www.arrow.com/en/products/stm32h523ceu6/stmicroelectronics?region=nac" (at 149.86 234.29 0)
+      (effects (font (size 1.27 1.27)) (justify left top) hide)
+    )
+    (property "Height" "0.6" (at 149.86 434.29 0)
+      (effects (font (size 1.27 1.27)) (justify left top) hide)
+    )
+    (property "Mouser Part Number" "511-STM32H523CEU6" (at 149.86 534.29 0)
+      (effects (font (size 1.27 1.27)) (justify left top) hide)
+    )
+    (property "Mouser Price/Stock" "https://www.mouser.co.uk/ProductDetail/STMicroelectronics/STM32H523CEU6?qs=ZcfC38r4Pot%2FWfU8ati%252BDA%3D%3D" (at 149.86 634.29 0)
+      (effects (font (size 1.27 1.27)) (justify left top) hide)
+    )
+    (property "Manufacturer_Name" "STMicroelectronics" (at 149.86 734.29 0)
+      (effects (font (size 1.27 1.27)) (justify left top) hide)
+    )
+    (property "Manufacturer_Part_Number" "STM32H523CEU6" (at 149.86 834.29 0)
+      (effects (font (size 1.27 1.27)) (justify left top) hide)
+    )
+    (pin "1")
+    (pin "10")
+    (pin "11")
+    (pin "12")
+    (pin "13")
+    (pin "14")
+    (pin "15")
+    (pin "16")
+    (pin "17")
+    (pin "18")
+    (pin "19")
+    (pin "2")
+    (pin "20")
+    (pin "21")
+    (pin "22")
+    (pin "23")
+    (pin "24")
+    (pin "25")
+    (pin "26")
+    (pin "27")
+    (pin "28")
+    (pin "29")
+    (pin "3")
+    (pin "30")
+    (pin "31")
+    (pin "32")
+    (pin "33")
+    (pin "34")
+    (pin "35")
+    (pin "36")
+    (pin "37")
+    (pin "38")
+    (pin "39")
+    (pin "4")
+    (pin "40")
+    (pin "41")
+    (pin "42")
+    (pin "43")
+    (pin "44")
+    (pin "45")
+    (pin "46")
+    (pin "47")
+    (pin "48")
+    (pin "49")
+    (pin "5")
+    (pin "6")
+    (pin "7")
+    (pin "8")
+    (pin "9")
+    (instances
+      (project "StrainGauge"
+        (path "/4f5fa9e6-e99a-4e4f-b2e1-754ea55be781"
+          (reference "IC1") (unit 1)
+        )
+      )
+    )
   )
   (sheet_instances
